File: 51.kicad_pcb (KiCad board)
At the start: 2 copper layers, 30.5 x 35.6 mm, 4 parts, among them J1 USB_C_Receptacle_USB2.0, J2 Conn_01x11, J3 Conn_01x11

Commit message: add switch */ /
Parts:
- removed STC15W204S: STC15W204S-35x-SOP16, Package_SO:STC_SOP-16_3.9x9.9mm_P1.27mm
- added C1: 47uF, Capacitor_SMD:C_0603_1608Metric, F.Cu at (106.1, 67.4)
- added C2: 0.1uF, Capacitor_SMD:C_0805_2012Metric, F.Cu at (108.5, 67.5)
- added D1: LED, LED_SMD:LED_1206_3216Metric, F.Cu at (120.2, 51.8)
- added D2: LED, LED_SMD:LED_1206_3216Metric, F.Cu at (104.4, 51.9)
- added R1: R, Resistor_SMD:R_0805_2012Metric, F.Cu at (120.2, 56.9)
- added R2: R, Resistor_SMD:R_0805_2012Metric, F.Cu at (104.4, 57.0)
- added SW1: SW_DPST, Button_Switch_THT:SW_Push_2P1T_Toggle_CK_PVA1xxH4xxxxxxV2, F.Cu at (109.3, 73.3)
- added U1: STC15W204S-35x-SOP16, Package_SO:STC_SOP-16_3.9x9.9mm_P1.27mm, F.Cu at (113.9, 64.4)
- moved J3 4.24 mm to (126.2, 53.3)
- moved J2 3.07 mm to (98.5, 53.3)
- moved J1 2.87 mm to (112.2, 53.0)
Connections:
- J2 pad 1: GND -> GND1
- J2 pad 10: +5V -> VCC
- J2 pad 11: GND -> GND1
- J2 pad 2: +5V -> VCC
- J3 pad 1: GND -> GND1
- J3 pad 10: +5V -> VCC
- J3 pad 11: GND -> GND1
- J3 pad 2: +5V -> VCC
Routing:
- net VCC: track 0.00 -> 101.8 mm, vias 0 -> 2
- net +5V: track 90.1 -> 51.6 mm, vias 0 -> 1
- net p3_1: track 8.83 -> 31.0 mm, vias 0 -> 2
- net p3_0: track 8.40 -> 26.4 mm, vias 0 -> 2
- net p1_5: track 7.77 -> 15.7 mm
- net p5_4: track 9.45 -> 17.1 mm
- net p1_4: track 7.77 -> 15.2 mm
- net p1_3: track 8.40 -> 14.7 mm
- net GND: track 5.63 -> 0.00 mm, vias 3 -> 0
- net p5_5: track 24.7 -> 19.4 mm, vias 0 -> 2
- net p1_2: track 8.83 -> 14.1 mm
- net GND1: track 0.00 -> 2.91 mm
- net Net-(D2-Pad2): track 0.00 -> 2.87 mm
- net Net-(D1-Pad2): track 0.00 -> 2.82 mm
- net p1_0: track 17.5 -> 19.8 mm
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- removed copper zone on B.Cu, net GND
- removed copper zone on F.Cu, net GND
Other:
- board size 30.5 x 35.6 mm -> 53.5 x 41.5 mm

Commit message: add cooper
Routing:
- added copper zone on B.Cu, net GND1
- added copper zone on F.Cu, net GND1
Changed lines of the file:
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@@
   (segment (start 120.2436 53.2922) (end 120.1674 53.216) (width 0.25) (layer "F.Cu") (net 19))
   (segment (start 104.4448 56.1359) (end 104.4448 53.2668) (width 0.25) (layer "F.Cu") (net 20))
-  (zone (net 0) (net_name "") (layers F&B.Cu "Edge.Cuts") (hatch edge 0.508)
+  (zone (net 18) (net_name "GND1") (layers F&B.Cu) (hatch edge 0.508)
     (connect_pads (clearance 0))
-    (min_thickness 0.254)
-    (keepout (tracks allowed) (vias allowed) (pads allowed) (copperpour allowed) (footprints allowed))
-    (fill (thermal_gap 0.508) (thermal_bridge_width 0.508))
+    (min_thickness 0.254) (filled_areas_thickness no)
+    (fill yes (thermal_gap 0.508) (thermal_bridge_width 0.508))
     (polygon
       (pts
-        (xy 135.6614 82.7786)
-        (xy 89.0778 82.8802)
-        (xy 89.4588 46.6852)
-        (xy 89.4334 46.6852)
-        (xy 135.89 46.5836)
+        (xy 135.9662 82.7278)
+        (xy 90.678 82.7278)
+        (xy 90.4748 47.244)
+        (xy 135.509 46.863)
       )
     )

Commit message: relayout
Parts:
- C1: footprint Capacitor_SMD:C_0603_1608Metric -> Capacitor_SMD:C_0805_2012Metric
- R1, R2: value R -> 10k
- moved SW1 34.8 mm to (93.1, 42.5)
- moved J3 25.2 mm to (108.2, 35.6)
- moved J1 24.5 mm to (95.5, 35.1)
- moved J2 22.7 mm to (84.3, 35.6)
- moved R1 22.2 mm to (98.6, 52.3), turned to 0 degrees
- moved U1 18.8 mm to (95.5, 60.5)
- moved C2 18.5 mm to (90.4, 63.5)
- moved C1 18.4 mm to (88.1, 63.5)
- moved D1 17.5 mm to (102.7, 52.3), turned to 180 degrees
- moved D2 14.5 mm to (89.9, 52.3), turned to 0 degrees
- moved R2 11.0 mm to (94.5, 52.3), turned to 0 degrees
Connections:
- J1 pad A5: GND -> unconnected-(J1-PadA5)
- J1 pad A6: GND -> unconnected-(J1-PadA6)
- J1 pad A7: GND -> unconnected-(J1-PadA7)
- J1 pad A8: GND -> unconnected-(J1-PadA8)
- J1 pad B5: GND -> unconnected-(J1-PadB5)
- J1 pad B6: GND -> unconnected-(J1-PadB6)
- J1 pad B7: GND -> unconnected-(J1-PadB7)
- J1 pad B8: GND -> unconnected-(J1-PadB8)
Routing:
- net +5V: track 51.6 -> 18.3 mm, vias 1 -> 0
- net VCC: track 101.8 -> 77.1 mm, vias 2 -> 0
- net GND: track 0.00 -> 23.7 mm
- net p5_5: track 19.4 -> 36.2 mm, vias 2 -> 1
- net p3_7: track 10.3 -> 24.7 mm, vias 0 -> 1
- net p3_6: track 10.0 -> 23.2 mm, vias 0 -> 1
- net p3_3: track 10.0 -> 21.5 mm, vias 0 -> 1
- net p3_2: track 10.5 -> 19.6 mm, vias 0 -> 1
- net p1_0: track 19.8 -> 26.8 mm, vias 2 -> 1
- net p1_2: track 14.1 -> 18.5 mm, vias 0 -> 1
- net p3_0: track 26.4 -> 30.5 mm, vias 2 -> 1
- net p5_4: track 17.1 -> 12.9 mm, vias 0 -> 1
- net p1_1: track 19.5 -> 23.4 mm, vias 2 -> 1
- net GND1: track 2.91 -> 0.00 mm
- net p1_3: track 14.7 -> 17.2 mm, vias 0 -> 1
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- removed copper zone on B.Cu, net GND1
Other:
- board size 53.5 x 41.5 mm -> 36.3 x 36.6 mm
- board text added: "STC15W204S"
