File: 51.kicad_sch (KiCad schematic)
At the start: 4 parts, among them J1 USB_C_Receptacle_USB2.0, J2 Conn_01x11, J3 Conn_01x11, U1 STC15W204S-35x-SOP16

Commit message: add switch */ /
Parts:
- added C1: 47uF, Capacitor_SMD:C_0603_1608Metric, symbol Device:C
- added C2: 0.1uF, Capacitor_SMD:C_0805_2012Metric, symbol Device:C
- added D1, D2: LED, LED_SMD:LED_1206_3216Metric, symbol Device:LED
- added R1, R2: R, Resistor_SMD:R_0805_2012Metric, symbol Device:R
- added SW1: SW_DPST, Button_Switch_THT:SW_Push_2P1T_Toggle_CK_PVA1xxH4xxxxxxV2, symbol Switch:SW_DPST
Connections:
- net +5V: now also SW1.3; no longer J2.10 (Pin_10), J2.2 (Pin_2), J3.10 (Pin_10), J3.2 (Pin_2), U1.6 (VCC)
- net GND: now also SW1.1; no longer J2.1 (Pin_1), J2.11 (Pin_11), J3.1 (Pin_1), J3.11 (Pin_11), U1.8 (GND)
- net p3_0: now also R1.1
- net p3_1: now also R2.2
- new net: D2.2 (A), R2.1
- new net: D1.2 (A), R1.2
- new net GND1: C1.2, C2.2, J2.1 (Pin_1), J2.11 (Pin_11), J3.1 (Pin_1), J3.11 (Pin_11), SW1.2, U1.8 (GND)
- new net VCC: C1.1, C2.1, D1.1 (K), D2.1 (K), J2.10 (Pin_10), J2.2 (Pin_2), J3.10 (Pin_10), J3.2 (Pin_2), SW1.4, U1.6 (VCC)
Other:
- moved on the sheet: J1, U1

Commit message: relayout
Parts:
- C1: footprint Capacitor_SMD:C_0603_1608Metric -> Capacitor_SMD:C_0805_2012Metric
- R1, R2: value R -> 10k
Connections:
- net GND: no longer J1.A5 (CC1), J1.A6 (D+), J1.A7 (D-), J1.A8 (SBU1), J1.B5 (CC2), J1.B6 (D+), J1.B7 (D-), J1.B8 (SBU2)
- net VCC: now also D1.2 (A), D2.2 (A); no longer D1.1 (K), D2.1 (K)
- net at R2.1: now also D2.1 (K); no longer D2.2 (A)
- net at R1.2: now also D1.1 (K); no longer D1.2 (A)
- no-connect marks 0 -> 8
Other:
- moved on the sheet: D1, D2
Changed lines of the file:
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@@
 (kicad_sch (version 20211123) (generator eeschema)
   (paper "A4")
-  (junction (at 48.895 118.11) (diameter 0) (color 0 0 0 0)
-  )
   (junction (at 97.79 103.505) (diameter 0) (color 0 0 0 0)
   )
-  (junction (at 48.895 105.41) (diameter 0) (color 0 0 0 0)
-  )
-  (junction (at 48.895 120.65) (diameter 0) (color 0 0 0 0)
-  )
-  (junction (at 48.895 97.79) (diameter 0) (color 0 0 0 0)
-  )
   (junction (at 48.895 128.27) (diameter 0) (color 0 0 0 0)
   )
@@
   (junction (at 98.425 111.125) (diameter 0) (color 0 0 0 0)
   )
-  (junction (at 48.895 107.95) (diameter 0) (color 0 0 0 0)
-  )
   (junction (at 33.655 128.27) (diameter 0) (color 0 0 0 0)
   )
-  (junction (at 48.895 110.49) (diameter 0) (color 0 0 0 0)
-  )
-  (junction (at 48.895 102.87) (diameter 0) (color 0 0 0 0)
-  )
   (junction (at 65.405 87.63) (diameter 0) (color 0 0 0 0)
   )
@@
   (junction (at 48.895 87.63) (diameter 0) (color 0 0 0 0)
   )
+  (no_connect (at 48.895 120.65))
+  (no_connect (at 48.895 118.11))
+  (no_connect (at 48.895 97.79))
+  (no_connect (at 48.895 95.25))
+  (no_connect (at 48.895 110.49))
+  (no_connect (at 48.895 107.95))
+  (no_connect (at 48.895 105.41))
+  (no_connect (at 48.895 102.87))
   (wire (pts (xy 68.58 128.27) (xy 83.185 128.27))
     (stroke (width 0) (type default) (color 0 0 0 0))
@@
     (stroke (width 0) (type default) (color 0 0 0 0))
   )
-  (wire (pts (xy 48.895 102.87) (xy 48.895 105.41))
-    (stroke (width 0) (type default) (color 0 0 0 0))
-  )
   (wire (pts (xy 108.585 33.02) (xy 115.57 33.02))
     (stroke (width 0) (type default) (color 0 0 0 0))
@@
     (stroke (width 0) (type default) (color 0 0 0 0))
   )
-  (wire (pts (xy 48.895 120.65) (xy 48.895 128.27))
-    (stroke (width 0) (type default) (color 0 0 0 0))
-  )
   (wire (pts (xy 100.965 111.125) (xy 103.505 111.125))
     (stroke (width 0) (type default) (color 0 0 0 0))
@@
     (stroke (width 0) (type default) (color 0 0 0 0))
   )
-  (wire (pts (xy 48.895 95.25) (xy 48.895 97.79))
-    (stroke (width 0) (type default) (color 0 0 0 0))
-  )
   (wire (pts (xy 93.345 103.505) (xy 93.345 104.775))
     (stroke (width 0) (type default) (color 0 0 0 0))
@@
     (stroke (width 0) (type default) (color 0 0 0 0))
   )
-  (wire (pts (xy 48.895 105.41) (xy 48.895 107.95))
-    (stroke (width 0) (type default) (color 0 0 0 0))
-  )
   (wire (pts (xy 123.19 127) (xy 175.26 127))
     (stroke (width 0) (type default) (color 0 0 0 0))
@@
     (stroke (width 0) (type default) (color 0 0 0 0))
   )
-  (wire (pts (xy 48.895 118.11) (xy 48.895 120.65))
-    (stroke (width 0) (type default) (color 0 0 0 0))
-  )
   (wire (pts (xy 113.03 103.505) (xy 122.555 103.505))
     (stroke (width 0) (type default) (color 0 0 0 0))
@@
     (stroke (width 0) (type default) (color 0 0 0 0))
   )
-  (wire (pts (xy 48.895 97.79) (xy 48.895 102.87))
-    (stroke (width 0) (type default) (color 0 0 0 0))
-  )
-  (wire (pts (xy 48.895 110.49) (xy 48.895 118.11))
-    (stroke (width 0) (type default) (color 0 0 0 0))
-  )
   (wire (pts (xy 48.895 90.17) (xy 48.895 87.63))
     (stroke (width 0) (type default) (color 0 0 0 0))
@@
   )
   (wire (pts (xy 48.895 128.27) (xy 68.58 128.27))
-    (stroke (width 0) (type default) (color 0 0 0 0))
-  )
-  (wire (pts (xy 48.895 107.95) (xy 48.895 110.49))
     (stroke (width 0) (type default) (color 0 0 0 0))
   )
@@
     (pin "1")
   )
-  (symbol (lib_id "Device:LED") (at 227.33 89.535 180) (unit 1)
-    (in_bom yes) (on_board yes) (fields_autoplaced)
-    (property "Reference" "D2" (id 0) (at 228.9175 82.55 0))
-    (property "Value" "LED" (id 1) (at 228.9175 85.09 0))
+  (symbol (lib_id "Device:LED") (at 227.33 89.535 0) (unit 1)
+    (in_bom yes) (on_board yes) (fields_autoplaced)
+    (property "Reference" "D2" (id 0) (at 225.7425 82.55 0))
+    (property "Value" "LED" (id 1) (at 225.7425 85.09 0))
     (property "Footprint" "LED_SMD:LED_1206_3216Metric" (id 2) (at 227.33 89.535 0)
       (effects (font (size 1.27 1.27)) hide)
@@
     (in_bom yes) (on_board yes)
     (property "Reference" "R1" (id 0) (at 215.9 67.945 90))
-    (property "Value" "R" (id 1) (at 215.9 70.485 90))
+    (property "Value" "10k" (id 1) (at 215.9 70.485 90))
     (property "Footprint" "Resistor_SMD:R_0805_2012Metric" (id 2) (at 215.9 75.438 90)
       (effects (font (size 1.27 1.27)) hide)
@@
     (pin "1")
   )
-  (symbol (lib_id "Device:LED") (at 223.52 73.66 180) (unit 1)
-    (in_bom yes) (on_board yes) (fields_autoplaced)
-    (property "Reference" "D1" (id 0) (at 225.1075 66.04 0))
-    (property "Value" "LED" (id 1) (at 225.1075 68.58 0))
+  (symbol (lib_id "Device:LED") (at 223.52 73.66 0) (unit 1)
+    (in_bom yes) (on_board yes) (fields_autoplaced)
+    (property "Reference" "D1" (id 0) (at 221.9325 67.31 0))
+    (property "Value" "LED" (id 1) (at 221.9325 69.85 0))
     (property "Footprint" "LED_SMD:LED_1206_3216Metric" (id 2) (at 223.52 73.66 0)
       (effects (font (size 1.27 1.27)) hide)
@@
       (effects (font (size 1.27 1.27)) (justify left))
     )
-    (property "Footprint" "Capacitor_SMD:C_0603_1608Metric" (id 2) (at 104.4702 111.125 0)
+    (property "Footprint" "Capacitor_SMD:C_0805_2012Metric" (id 2) (at 104.4702 111.125 0)
       (effects (font (size 1.27 1.27)) hide)
     )
@@
   (symbol (lib_id "Device:R") (at 219.71 89.535 270) (unit 1)
     (in_bom yes) (on_board yes) (fields_autoplaced)
-    (property "Reference" "R2" (id 0) (at 219.71 83.185 90))
-    (property "Value" "R" (id 1) (at 219.71 85.725 90))
+    (property "Reference" "R2" (id 0) (at 219.71 83.82 90))
+    (property "Value" "10k" (id 1) (at 219.71 86.36 90))
     (property "Footprint" "Resistor_SMD:R_0805_2012Metric" (id 2) (at 219.71 87.757 90)
       (effects (font (size 1.27 1.27)) hide)
@@
     )
     (path "/ea1253fa-1698-43d3-92ec-7b4c87043781"
-      (reference "C1") (unit 1) (value "47uF") (footprint "Capacitor_SMD:C_0603_1608Metric")
+      (reference "C1") (unit 1) (value "47uF") (footprint "Capacitor_SMD:C_0805_2012Metric")
     )
     (path "/7c587ae8-ad17-491e-909a-5c161db9f920"
@@
     )
     (path "/852aaec7-ebf7-4120-b477-769cc871567a"
-      (reference "R1") (unit 1) (value "R") (footprint "Resistor_SMD:R_0805_2012Metric")
+      (reference "R1") (unit 1) (value "10k") (footprint "Resistor_SMD:R_0805_2012Metric")
     )
     (path "/eb1ca729-ba13-4857-84a3-2f88e486b697"
-      (reference "R2") (unit 1) (value "R") (footprint "Resistor_SMD:R_0805_2012Metric")
+      (reference "R2") (unit 1) (value "10k") (footprint "Resistor_SMD:R_0805_2012Metric")
     )
     (path "/1e378bd9-6d2c-473f-95bb-e0afe58cd0e3"
